File: LED_Coaster.kicad_sch (KiCad schematic)
At the start: 60 parts, among them J1 USB_C_Receptacle_USB2.0, SW1 SW_Push, SW2 SW_DIP_x01, SW3 SW_DIP_x01, U1 ATmega32U4-A, Y1 Crystal_GND24

Commit message: Added more components
Parts:
- removed C1: 1uF, Capacitor_SMD:C_0805_2012Metric_Pad1.18x1.45mm_HandSolder, symbol Device:C
- removed C2: 10uF, Capacitor_SMD:C_0805_2012Metric_Pad1.18x1.45mm_HandSolder, symbol Device:C
- removed C3, C4, C5: 0.1uF, Capacitor_SMD:C_0805_2012Metric_Pad1.18x1.45mm_HandSolder, symbol Device:C
- removed C6, C7: 22pF, Capacitor_SMD:C_0805_2012Metric_Pad1.18x1.45mm_HandSolder, symbol Device:C
- removed D33: LED, LED_SMD:LED_0805_2012Metric_Pad1.15x1.40mm_HandSolder, symbol Device:LED
- removed R1, R4: 10K, Resistor_SMD:R_0805_2012Metric_Pad1.20x1.40mm_HandSolder, symbol Device:R
- removed R2, R3: 22, Resistor_SMD:R_0805_2012Metric_Pad1.20x1.40mm_HandSolder, symbol Device:R
- removed R5, R6: 5.1K, Resistor_SMD:R_0805_2012Metric_Pad1.20x1.40mm_HandSolder, symbol Device:R
- removed R9: 150, Resistor_SMD:R_0805_2012Metric_Pad1.20x1.40mm_HandSolder, symbol Device:R
- removed SW1: SW_Push, Button_Switch_SMD:SW_SPST_SKQG_WithoutStem, symbol Switch:SW_Push
- removed U1: ATmega32U4-A, Package_QFP:TQFP-44_10x10mm_P0.8mm, symbol MCU_Microchip_ATmega:ATmega32U4-A
- removed Y1: Crystal_GND24, Crystal:Crystal_SMD_3225-4Pin_3.2x2.5mm_HandSoldering, symbol Device:Crystal_GND24
- added BT1: Battery_Cell, Battery:Battery_Panasonic_CR2032-HFN_Horizontal_CircularHoles, symbol Device:Battery_Cell
- added EMB1: ~, Library:EMB1082, symbol New_Library:EMB1082
- added J2: Conn_ARM_SWD_TagConnect_TC2030-NL, Connector:Tag-Connect_TC2030-IDC-NL_2x03_P1.27mm_Vertical, symbol Connector:Conn_ARM_SWD_TagConnect_TC2030-NL
- added U2: LD1117S33TR_SOT223, Package_TO_SOT_SMD:SOT-223-3_TabPin2, symbol Regulator_Linear:LD1117S33TR_SOT223
Connections:
- net +5V: now also U2.3 (VI)
- net GND: now also EMB1.9 (GND), J2.5 (GND), U2.1 (GND)
- net large_ring: now also EMB1.19 (P0_1)
- net small_ring: now also EMB1.20 (P0_0)
- net D+: no longer names the net of J1.A6 (D+)
- net D+: no longer J1.B6 (D+)
- net D-: no longer names the net of J1.A7 (D-)
- net D-: no longer J1.B7 (D-)
- new net: EMB1.17 (SWD_IO), J2.2 (SWDIO)
- new net: EMB1.1 (#RESET), J2.3 (~{RESET})
- new net: EMB1.18 (SWD_CLK), J2.4 (SWCLK)
- new net 3.3V: EMB1.8 (VDD3V3), J2.1 (VCC), U2.2 (VO)
- no-connect marks 27 -> 4

Commit message: Added traces for EMB1082 and power switch
Parts:
- removed BT1: Battery_Cell, Battery:Battery_Panasonic_CR2032-HFN_Horizontal_CircularHoles, symbol Device:Battery_Cell
- removed F1: Polyfuse, Fuse:Fuse_1206_3216Metric_Pad1.42x1.75mm_HandSolder, symbol Device:Polyfuse
- removed J1: USB_C_Receptacle_USB2.0, Connector_USB:USB_C_Receptacle_HRO_TYPE-C-31-M-12, symbol Connector:USB_C_Receptacle_USB2.0
- added D33: LED, LED_SMD:LED_0805_2012Metric_Pad1.15x1.40mm_HandSolder, symbol Device:LED
- added R1: 150, Resistor_SMD:R_0805_2012Metric_Pad1.20x1.40mm_HandSolder, symbol Device:R
- added SW1: SW_DIP_x01, Button_Switch_SMD:SW_SPDT_PCM12, symbol Switch:SW_DIP_x01
- added TP1, TP2: TestPoint, TestPoint:TestPoint_Loop_D1.80mm_Drill1.0mm_Beaded, symbol Connector:TestPoint
Connections:
- net +5V: now also R1.2, SW1.2
- net GND: now also D33.1 (K), TP2.1
- new net: D33.2 (A), R1.1
- new net: SW1.1, TP1.1
- no-connect marks 4 -> 2
